File: hardware/untitled.sch (EAGLE design)
At the start: 39 parts, among them J1 AUDIO_JACK_TRRSSMD_RA, U1 AT32UC3A1512/1256/1128, U2 USD-SOCKETUSD, Y2 CRYSTAL-GROUNDEDSMD-5X3.2

Commit message: PCB updated
Parts:
- added C10, C8: 22 pF, rcl:C-EUC0603
- added C22, C9: 33n, rcl:C-EUC0402
- added J2: GT-USB-7010, GT-USB-7010:GT-USB-7010
- added R2: 10k, rcl:R-EU_R0402
- added U$3, U$8: SMT3X6X3.5MM, mw:SMT3X6X3.5MM
- added Y1: CRYSTAL-GROUNDEDSMD-5X3.2, SparkFun-Clocks:CRYSTAL-GROUNDEDSMD-5X3.2
- C1: device rcl:CPOL-EUSMCB -> rcl:CPOL-EUSMCA
- C2, C3, C4, C5: value (none) -> 2n7
- C6, C7: value (none) -> 33n
Connections:
- new net D_N: J2.A7/DN1, J2.B7/DN2, U1.DM
- new net D_P: J2.A6/DP1, J2.B6/DP2, U1.DP
- new net KEY_VOLUP: U$8.B, U1.PWM-PWM[4]/USART1-RXD/PA05
- new net OSC_IN: C10.1, U1.PC02/XIN0, Y1.2
- new net OSC_OUT: C8.1, U1.PC03/XOUT0, Y1.1
- new net VBUS: J2.A4/B9/VBUS, J2.B4/A9/VBUS, U1.VBUS
- net 3V: now also R2.2
- net GND: now also C10.2, C22.2, C8.2, C9.2, J2.A1/B12/GND, J2.B1/A12/GND, U$8.A, U$8.MNT, Y1.3
- net MOSI: now also R2.1
- net VDDCORE: now also C22.1, C9.1
Other:
- moved on the sheet: C5

Commit message: PCB updated
Parts:
- removed J2: GT-USB-7010, GT-USB-7010:GT-USB-7010
- added C27: 2n7, rcl:C-EUC0402
- added C28: 33n, rcl:C-EUC0402
- added R3, R4, R7: (no value), rcl:R-EU_R0402
- added U$4: MICRO-USBV2, microusb:MICRO-USBV2
- R15: device rcl:R-EU_R0603 -> rcl:R-EU_R0402
Connections:
- new net D_P_1: R7.2, U$4.D+
- new net N$4: R4.2, U$4.D-
- net 3V: now also C27.1, C28.1, R3.2
- net D_N: now also R4.1; no longer J2.A7/DN1, J2.B7/DN2
- net D_P: now also R7.1; no longer J2.A6/DP1, J2.B6/DP2
- net GND: now also C27.2, C28.2, U$4.GND; no longer J2.A1/B12/GND, J2.B1/A12/GND
- net I2C1_SDA: now also R3.1
- net VBUS: now also U$4.VCC; no longer J2.A4/B9/VBUS, J2.B4/A9/VBUS
Changed lines of the file:
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@@
 <part name="C23" library="rcl" deviceset="CPOL-EU" device="SMCE"/>
 <part name="C24" library="rcl" deviceset="CPOL-EU" device="SMCE"/>
-<part name="R15" library="rcl" deviceset="R-EU_" device="R0603"/>
+<part name="R15" library="rcl" deviceset="R-EU_" device="R0402"/>
 <part name="C25" library="rcl" deviceset="C-EU" device="C0603" value="1u"/>
 <part name="C26" library="rcl" deviceset="C-EU" device="C0603" value="220p"/>
@@
 <part name="GND13" library="supply1" deviceset="GND" device=""/>
 <part name="U$3" library="mw" deviceset="SMT3X6X3.5MM" device=""/>
-<part name="J2" library="GT-USB-7010" deviceset="GT-USB-7010" device=""/>
+<part name="R4" library="rcl" deviceset="R-EU_" device="R0402"/>
+<part name="U$4" library="microusb" deviceset="MICRO-USB" device="V2"/>
+<part name="R7" library="rcl" deviceset="R-EU_" device="R0402"/>
+<part name="GND16" library="supply1" deviceset="GND" device=""/>
+<part name="C27" library="rcl" deviceset="C-EU" device="C0402" value="2n7"/>
+<part name="GND14" library="supply1" deviceset="GND" device=""/>
+<part name="C28" library="rcl" deviceset="C-EU" device="C0402" value="33n"/>
+<part name="GND15" library="supply1" deviceset="GND" device=""/>
+<part name="R3" library="rcl" deviceset="R-EU_" device="R0402"/>
 </parts>
 <sheets>
@@
 <instance part="GND13" gate="1" x="284.48" y="139.7"/>
 <instance part="U$3" gate="G$1" x="259.08" y="200.66"/>
-<instance part="J2" gate="G$1" x="25.4" y="-101.6"/>
+<instance part="R4" gate="G$1" x="124.46" y="-88.9" rot="R180"/>
+<instance part="U$4" gate="G$1" x="96.52" y="-86.36"/>
+<instance part="R7" gate="G$1" x="124.46" y="-96.52" rot="R180"/>
+<instance part="GND16" gate="1" x="114.3" y="-104.14"/>
+<instance part="C27" gate="G$1" x="-58.42" y="27.94"/>
+<instance part="GND14" gate="1" x="-58.42" y="17.78"/>
+<instance part="C28" gate="G$1" x="-66.04" y="27.94"/>
+<instance part="GND15" gate="1" x="-66.04" y="17.78"/>
+<instance part="R3" gate="G$1" x="243.84" y="-5.08" rot="R90"/>
 </instances>
 <busses>
@@
 </segment>
 <segment>
-<pinref part="J2" gate="G$1" pin="A1/B12/GND"/>
-<wire x1="2.54" y1="-93.98" x2="0" y2="-93.98" width="0.1524" layer="91"/>
-<wire x1="0" y1="-93.98" x2="0" y2="-83.82" width="0.1524" layer="91"/>
-<wire x1="0" y1="-83.82" x2="0" y2="-78.74" width="0.1524" layer="91"/>
-<wire x1="0" y1="-83.82" x2="55.88" y2="-83.82" width="0.1524" layer="91"/>
-<wire x1="55.88" y1="-83.82" x2="55.88" y2="-93.98" width="0.1524" layer="91"/>
-<junction x="0" y="-83.82"/>
-<pinref part="J2" gate="G$1" pin="B1/A12/GND"/>
-<wire x1="55.88" y1="-93.98" x2="50.8" y2="-93.98" width="0.1524" layer="91"/>
+<pinref part="U$4" gate="G$1" pin="GND"/>
+<pinref part="GND16" gate="1" pin="GND"/>
+<wire x1="111.76" y1="-99.06" x2="114.3" y2="-99.06" width="0.1524" layer="91"/>
+<wire x1="114.3" y1="-99.06" x2="114.3" y2="-101.6" width="0.1524" layer="91"/>
+</segment>
+<segment>
+<pinref part="C27" gate="G$1" pin="2"/>
+<pinref part="GND14" gate="1" pin="GND"/>
+<wire x1="-58.42" y1="20.32" x2="-58.42" y2="22.86" width="0.1524" layer="91"/>
+</segment>
+<segment>
+<pinref part="C28" gate="G$1" pin="2"/>
+<pinref part="GND15" gate="1" pin="GND"/>
+<wire x1="-66.04" y1="20.32" x2="-66.04" y2="22.86" width="0.1524" layer="91"/>
 </segment>
 </net>
@@
 <segment>
 <pinref part="R15" gate="G$1" pin="2"/>
-<wire x1="238.76" y1="0" x2="238.76" y2="5.08" width="0.1524" layer="91"/>
+<wire x1="238.76" y1="0" x2="238.76" y2="2.54" width="0.1524" layer="91"/>
 <label x="238.76" y="5.08" size="1.4224" layer="95" rot="R90" xref="yes"/>
+<pinref part="R3" gate="G$1" pin="2"/>
+<wire x1="238.76" y1="2.54" x2="238.76" y2="5.08" width="0.1524" layer="91"/>
+<wire x1="238.76" y1="2.54" x2="243.84" y2="2.54" width="0.1524" layer="91"/>
+<wire x1="243.84" y1="2.54" x2="243.84" y2="0" width="0.1524" layer="91"/>
+<junction x="238.76" y="2.54"/>
 </segment>
 <segment>
@@
 </segment>
 <segment>
+<pinref part="U1" gate="G$1" pin="ADVREF"/>
+<wire x1="-15.24" y1="22.86" x2="-30.48" y2="22.86" width="0.1524" layer="91"/>
+</segment>
+<segment>
+<pinref part="C27" gate="G$1" pin="1"/>
+<wire x1="-58.42" y1="38.1" x2="-58.42" y2="30.48" width="0.1524" layer="91"/>
+<pinref part="C28" gate="G$1" pin="1"/>
+<wire x1="-58.42" y1="38.1" x2="-66.04" y2="38.1" width="0.1524" layer="91"/>
+<wire x1="-66.04" y1="38.1" x2="-66.04" y2="30.48" width="0.1524" layer="91"/>
+<junction x="-58.42" y="38.1"/>
 <pinref part="U1" gate="G$1" pin="VDDIO@79"/>
 <wire x1="-15.24" y1="27.94" x2="-17.78" y2="27.94" width="0.1524" layer="91"/>
@@
 <wire x1="-17.78" y1="17.78" x2="-17.78" y2="27.94" width="0.1524" layer="91"/>
 <junction x="-17.78" y="27.94"/>
-</segment>
-<segment>
-<pinref part="U1" gate="G$1" pin="ADVREF"/>
-<wire x1="-15.24" y1="22.86" x2="-30.48" y2="22.86" width="0.1524" layer="91"/>
+<wire x1="-58.42" y1="38.1" x2="-17.78" y2="38.1" width="0.1524" layer="91"/>
+<junction x="-17.78" y="38.1"/>
 </segment>
 </net>
@@
 <segment>
 <pinref part="U$2" gate="G$1" pin="SDIN"/>
-<wire x1="266.7" y1="-17.78" x2="235.712" y2="-17.78" width="0.1524" layer="91"/>
+<wire x1="266.7" y1="-17.78" x2="243.84" y2="-17.78" width="0.1524" layer="91"/>
 <label x="235.712" y="-17.78" size="1.4224" layer="95" rot="R180" xref="yes"/>
+<pinref part="R3" gate="G$1" pin="1"/>
+<wire x1="243.84" y1="-17.78" x2="235.712" y2="-17.78" width="0.1524" layer="91"/>
+<wire x1="243.84" y1="-10.16" x2="243.84" y2="-17.78" width="0.1524" layer="91"/>
+<junction x="243.84" y="-17.78"/>
 </segment>
 <segment>
@@
 <net name="D_P" class="0">
 <segment>
-<pinref part="J2" gate="G$1" pin="A6/DP1"/>
-<wire x1="2.54" y1="-101.6" x2="-2.54" y2="-101.6" width="0.1524" layer="91"/>
-<wire x1="-2.54" y1="-101.6" x2="-2.54" y2="-114.3" width="0.1524" layer="91"/>
-<wire x1="-2.54" y1="-114.3" x2="-2.54" y2="-119.38" width="0.1524" layer="91"/>
-<wire x1="-2.54" y1="-114.3" x2="55.88" y2="-114.3" width="0.1524" layer="91"/>
-<wire x1="55.88" y1="-114.3" x2="55.88" y2="-104.14" width="0.1524" layer="91"/>
-<junction x="-2.54" y="-114.3"/>
-<pinref part="J2" gate="G$1" pin="B6/DP2"/>
-<wire x1="55.88" y1="-104.14" x2="50.8" y2="-104.14" width="0.1524" layer="91"/>
-</segment>
-<segment>
 <pinref part="U1" gate="G$1" pin="DP"/>
 <wire x1="-15.24" y1="104.14" x2="-22.86" y2="104.14" width="0.1524" layer="91"/>
 </segment>
+<segment>
+<pinref part="R7" gate="G$1" pin="1"/>
+<wire x1="129.54" y1="-96.52" x2="132.08" y2="-96.52" width="0.1524" layer="91"/>
+</segment>
 </net>
 <net name="D_N" class="0">
-<segment>
-<pinref part="J2" gate="G$1" pin="A7/DN1"/>
-<wire x1="2.54" y1="-104.14" x2="0" y2="-104.14" width="0.1524" layer="91"/>
-<wire x1="0" y1="-104.14" x2="0" y2="-116.84" width="0.1524" layer="91"/>
-<wire x1="0" y1="-119.38" x2="0" y2="-116.84" width="0.1524" layer="91"/>
-<wire x1="0" y1="-116.84" x2="58.42" y2="-116.84" width="0.1524" layer="91"/>
-<wire x1="58.42" y1="-116.84" x2="58.42" y2="-101.6" width="0.1524" layer="91"/>
-<junction x="0" y="-116.84"/>
-<pinref part="J2" gate="G$1" pin="B7/DN2"/>
-<wire x1="58.42" y1="-101.6" x2="50.8" y2="-101.6" width="0.1524" layer="91"/>
-</segment>
 <segment>
 <pinref part="U1" gate="G$1" pin="DM"/>
 <wire x1="-15.24" y1="109.22" x2="-22.86" y2="109.22" width="0.1524" layer="91"/>
 </segment>
+<segment>
+<pinref part="R4" gate="G$1" pin="1"/>
+<wire x1="129.54" y1="-88.9" x2="132.08" y2="-88.9" width="0.1524" layer="91"/>
+</segment>
 </net>
 <net name="VBUS" class="0">
@@
 </segment>
 <segment>
-<pinref part="J2" gate="G$1" pin="A4/B9/VBUS"/>
-<wire x1="2.54" y1="-96.52" x2="-2.54" y2="-96.52" width="0.1524" layer="91"/>
-<wire x1="-2.54" y1="-96.52" x2="-2.54" y2="-86.36" width="0.1524" layer="91"/>
-<wire x1="-2.54" y1="-86.36" x2="-2.54" y2="-78.74" width="0.1524" layer="91"/>
-<wire x1="-2.54" y1="-86.36" x2="58.42" y2="-86.36" width="0.1524" layer="91"/>
-<wire x1="58.42" y1="-86.36" x2="58.42" y2="-96.52" width="0.1524" layer="91"/>
-<junction x="-2.54" y="-86.36"/>
-<pinref part="J2" gate="G$1" pin="B4/A9/VBUS"/>
-<wire x1="58.42" y1="-96.52" x2="50.8" y2="-96.52" width="0.1524" layer="91"/>
-</segment>
-</net>
+<pinref part="U$4" gate="G$1" pin="VCC"/>
+<wire x1="111.76" y1="-88.9" x2="114.3" y2="-88.9" width="0.1524" layer="91"/>
+<wire x1="114.3" y1="-88.9" x2="114.3" y2="-81.28" width="0.1524" layer="91"/>
+</segment>
+</net>
+<net name="N$4" class="0">
+<segment>
+<pinref part="R4" gate="G$1" pin="2"/>
+<pinref part="U$4" gate="G$1" pin="D-"/>
+<wire x1="119.38" y1="-88.9" x2="116.84" y2="-88.9" width="0.1524" layer="91"/>
+<wire x1="116.84" y1="-88.9" x2="116.84" y2="-91.44" width="0.1524" layer="91"/>
+<wire x1="116.84" y1="-91.44" x2="111.76" y2="-91.44" width="0.1524" layer="91"/>
+</segment>
+</net>
+<net name="D_P_1" class="0">
+<segment>
+<pinref part="R7" gate="G$1" pin="2"/>
+<wire x1="116.84" y1="-96.52" x2="119.38" y2="-96.52" width="0.1524" layer="91"/>
+<pinref part="U$4" gate="G$1" pin="D+"/>
+<wire x1="111.76" y1="-93.98" x2="116.84" y2="-93.98" width="0.1524" layer="91"/>
+<wire x1="116.84" y1="-93.98" x2="116.84" y2="-96.52" width="0.1524" layer="91"/>
+</segment>
+</net>

Commit message: PCB updated
Parts:
- added C30, C32: 33n, rcl:C-EUC0402
- added C31, C33: 100n, rcl:C-EUC0402
- C27: value 2n7 -> 33n
- C28: value 33n -> 100n
Connections:
- net 3V: now also C30.1, C31.1, C32.1, C33.1
- net GND: now also C30.2, C31.2, C32.2, C33.2
Other:
- moved on the sheet: C27, C28
Changed lines of the file:
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@@
 <part name="R7" library="rcl" deviceset="R-EU_" device="R0402"/>
 <part name="GND16" library="supply1" deviceset="GND" device=""/>
-<part name="C27" library="rcl" deviceset="C-EU" device="C0402" value="2n7"/>
+<part name="C27" library="rcl" deviceset="C-EU" device="C0402" value="33n"/>
 <part name="GND14" library="supply1" deviceset="GND" device=""/>
-<part name="C28" library="rcl" deviceset="C-EU" device="C0402" value="33n"/>
+<part name="C28" library="rcl" deviceset="C-EU" device="C0402" value="100n"/>
 <part name="GND15" library="supply1" deviceset="GND" device=""/>
 <part name="R3" library="rcl" deviceset="R-EU_" device="R0402"/>
+<part name="C30" library="rcl" deviceset="C-EU" device="C0402" value="33n"/>
+<part name="GND22" library="supply1" deviceset="GND" device=""/>
+<part name="C31" library="rcl" deviceset="C-EU" device="C0402" value="100n"/>
+<part name="GND25" library="supply1" deviceset="GND" device=""/>
+<part name="C32" library="rcl" deviceset="C-EU" device="C0402" value="33n"/>
+<part name="GND26" library="supply1" deviceset="GND" device=""/>
+<part name="C33" library="rcl" deviceset="C-EU" device="C0402" value="100n"/>
+<part name="GND27" library="supply1" deviceset="GND" device=""/>
 </parts>
 <sheets>
@@
 <instance part="R7" gate="G$1" x="124.46" y="-96.52" rot="R180"/>
 <instance part="GND16" gate="1" x="114.3" y="-104.14"/>
-<instance part="C27" gate="G$1" x="-58.42" y="27.94"/>
-<instance part="GND14" gate="1" x="-58.42" y="17.78"/>
-<instance part="C28" gate="G$1" x="-66.04" y="27.94"/>
-<instance part="GND15" gate="1" x="-66.04" y="17.78"/>
+<instance part="C27" gate="G$1" x="-88.9" y="27.94"/>
+<instance part="GND14" gate="1" x="-88.9" y="17.78"/>
+<instance part="C28" gate="G$1" x="-96.52" y="27.94"/>
+<instance part="GND15" gate="1" x="-96.52" y="17.78"/>
 <instance part="R3" gate="G$1" x="243.84" y="-5.08" rot="R90"/>
+<instance part="C30" gate="G$1" x="-73.66" y="27.94"/>
+<instance part="GND22" gate="1" x="-73.66" y="17.78"/>
+<instance part="C31" gate="G$1" x="-81.28" y="27.94"/>
+<instance part="GND25" gate="1" x="-81.28" y="17.78"/>
+<instance part="C32" gate="G$1" x="-58.42" y="27.94"/>
+<instance part="GND26" gate="1" x="-58.42" y="17.78"/>
+<instance part="C33" gate="G$1" x="-66.04" y="27.94"/>
+<instance part="GND27" gate="1" x="-66.04" y="17.78"/>
 </instances>
 <busses>
@@
 <pinref part="C27" gate="G$1" pin="2"/>
 <pinref part="GND14" gate="1" pin="GND"/>
-<wire x1="-58.42" y1="20.32" x2="-58.42" y2="22.86" width="0.1524" layer="91"/>
+<wire x1="-88.9" y1="20.32" x2="-88.9" y2="22.86" width="0.1524" layer="91"/>
 </segment>
 <segment>
 <pinref part="C28" gate="G$1" pin="2"/>
 <pinref part="GND15" gate="1" pin="GND"/>
+<wire x1="-96.52" y1="20.32" x2="-96.52" y2="22.86" width="0.1524" layer="91"/>
+</segment>
+<segment>
+<pinref part="C30" gate="G$1" pin="2"/>
+<pinref part="GND22" gate="1" pin="GND"/>
+<wire x1="-73.66" y1="20.32" x2="-73.66" y2="22.86" width="0.1524" layer="91"/>
+</segment>
+<segment>
+<pinref part="C31" gate="G$1" pin="2"/>
+<pinref part="GND25" gate="1" pin="GND"/>
+<wire x1="-81.28" y1="20.32" x2="-81.28" y2="22.86" width="0.1524" layer="91"/>
+</segment>
+<segment>
+<pinref part="C32" gate="G$1" pin="2"/>
+<pinref part="GND26" gate="1" pin="GND"/>
+<wire x1="-58.42" y1="20.32" x2="-58.42" y2="22.86" width="0.1524" layer="91"/>
+</segment>
+<segment>
+<pinref part="C33" gate="G$1" pin="2"/>
+<pinref part="GND27" gate="1" pin="GND"/>
 <wire x1="-66.04" y1="20.32" x2="-66.04" y2="22.86" width="0.1524" layer="91"/>
 </segment>
@@
 <segment>
 <pinref part="C27" gate="G$1" pin="1"/>
-<wire x1="-58.42" y1="38.1" x2="-58.42" y2="30.48" width="0.1524" layer="91"/>
+<wire x1="-88.9" y1="38.1" x2="-88.9" y2="30.48" width="0.1524" layer="91"/>
 <pinref part="C28" gate="G$1" pin="1"/>
-<wire x1="-58.42" y1="38.1" x2="-66.04" y2="38.1" width="0.1524" layer="91"/>
-<wire x1="-66.04" y1="38.1" x2="-66.04" y2="30.48" width="0.1524" layer="91"/>
-<junction x="-58.42" y="38.1"/>
+<wire x1="-88.9" y1="38.1" x2="-96.52" y2="38.1" width="0.1524" layer="91"/>
+<wire x1="-96.52" y1="38.1" x2="-96.52" y2="30.48" width="0.1524" layer="91"/>
+<junction x="-88.9" y="38.1"/>
 <pinref part="U1" gate="G$1" pin="VDDIO@79"/>
 <wire x1="-15.24" y1="27.94" x2="-17.78" y2="27.94" width="0.1524" layer="91"/>
@@
 <wire x1="-17.78" y1="17.78" x2="-17.78" y2="27.94" width="0.1524" layer="91"/>
 <junction x="-17.78" y="27.94"/>
+<wire x1="-88.9" y1="38.1" x2="-81.28" y2="38.1" width="0.1524" layer="91"/>
+<junction x="-17.78" y="38.1"/>
+<pinref part="C31" gate="G$1" pin="1"/>
+<wire x1="-81.28" y1="38.1" x2="-73.66" y2="38.1" width="0.1524" layer="91"/>
+<wire x1="-73.66" y1="38.1" x2="-66.04" y2="38.1" width="0.1524" layer="91"/>
+<wire x1="-66.04" y1="38.1" x2="-58.42" y2="38.1" width="0.1524" layer="91"/>
 <wire x1="-58.42" y1="38.1" x2="-17.78" y2="38.1" width="0.1524" layer="91"/>
-<junction x="-17.78" y="38.1"/>
+<wire x1="-81.28" y1="30.48" x2="-81.28" y2="38.1" width="0.1524" layer="91"/>
+<junction x="-81.28" y="38.1"/>
+<pinref part="C30" gate="G$1" pin="1"/>
+<wire x1="-73.66" y1="30.48" x2="-73.66" y2="38.1" width="0.1524" layer="91"/>
+<junction x="-73.66" y="38.1"/>
+<pinref part="C33" gate="G$1" pin="1"/>
+<wire x1="-66.04" y1="30.48" x2="-66.04" y2="38.1" width="0.1524" layer="91"/>
+<junction x="-66.04" y="38.1"/>
+<pinref part="C32" gate="G$1" pin="1"/>
+<wire x1="-58.42" y1="30.48" x2="-58.42" y2="38.1" width="0.1524" layer="91"/>
+<junction x="-58.42" y="38.1"/>
 </segment>
 </net>

Commit message: PCB update. USB-C instead of microUSB, PMIC (work in progress)
Parts:
- removed C10, C11, C12: 22 pF, rcl:C-EUC0603
- removed U$4: MICRO-USBV2, microusb:MICRO-USBV2
- removed Y1, Y2: CRYSTAL-GROUNDEDSMD-5X3.2, SparkFun-Clocks:CRYSTAL-GROUNDEDSMD-5X3.2
- added J2: USB4110-GF-A, connector_tst:USB4110-GF-A
- added JP1: (no value), pinhead:PINHD-2X5
- added L2: COILCRAFT-LPS4018, passives:COILCRAFT-LPS4018
- added R10, R11, R5, R6, R8, R9: (no value), rcl:R-EU_R0402
- added U$5, U$6: ASE, crystal:ASE
- added U3: LTC3558EUDTRPBFQFN-20_UD_LIT-M, mw:LTC3558EUDTRPBFQFN-20_UD_LIT-M
- C20: device rcl:C-EUC0603 -> rcl:C-EUC0402
- C8: value 22 pF -> (none)
Connections:
- removed net D_P_1: R7.2, U$4.D+
- removed net N$4: R4.2, U$4.D-
- removed net XTI: C11.1, U$2.XTI/MCLK, Y2.1
- removed net XTO: C12.1, U$2.XTO, Y2.2
- new net /RESET: JP1.6, U1.!RESET
- new net D2_N: J2.DN1, J2.DN2, R4.2
- new net D2_P: J2.DP1, J2.DP2, R7.2
- new net MCLK: U$2.XTI/MCLK, U$6.OUT
- new net N$10: JP1.8
- new net N$2: L2.2, U3.SWAB2
- new net N$3: L2.1, U3.SWCD2
- new net N$5: R5.2, U3.PROG
- new net N$6: R6.2, U3.FB1
- new net N$7: R8.2, R9.1, U3.FB2
- new net N$8: J2.CC2, R11.2
- new net N$9: J2.CC1, R10.2
- new net TCK: JP1.1, U1.TCK
- new net TDI: JP1.9, U1.TDI
- new net TDO: JP1.3, U1.TDO
- new net TMS: JP1.5, U1.TMS
- net 3V: now also C8.1, JP1.4, R9.2, U$5.VDD, U$6.VDD, U3.VOUT2; no longer U1.VDDIN
- net GND: now also J2.GND, JP1.10, JP1.2, R10.1, R11.1, R5.1, R6.1, R8.1, U$5.GND, U$6.GND, U1.VDDIN, U1.VDDOUT, U3.SUSP; no longer C10.2, C11.2, C12.2, U$4.GND, Y1.3, Y2.3
- net OSC_IN: now also U$5.OUT; no longer C10.1, Y1.2
- net OSC_OUT: no longer C8.1, Y1.1
- net VBUS: now also J2.VBUS, U3.VCC; no longer U$4.VCC
- net VDDCORE: no longer U1.VDDOUT
Other:
- moved on the sheet: C19, C20, C21, C8, R4, R7

Commit message: MCU moved right to make place for PMIC
Parts:
- C8: device rcl:C-EUC0603 -> rcl:C-EUC0402
Changed lines of the file:
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@@
 <part name="U$6" library="crystal" deviceset="ASE" device=""/>
 <part name="GND30" library="supply1" deviceset="GND" device=""/>
-<part name="C8" library="rcl" deviceset="C-EU" device="C0603"/>
+<part name="C8" library="rcl" deviceset="C-EU" device="C0402"/>
 <part name="GND18" library="supply1" deviceset="GND" device=""/>
 <part name="J2" library="connector_tst" deviceset="USB4110-GF-A" device=""/>
